File: extensions/BreakoutTerm/BreakoutTerm.kicad_pcb (KiCad board)
At the start: 2 copper layers, 37 x 28.5 mm, 7 parts, among them M1 MH_3.2mm, M2 MH_3.2mm, P1 *, P2 CONN_01X10, P3 *

Commit message: Corrected part number for gadgeteer connectors; update libraries; add some doc files
Parts:
- P1, P3: footprint SBV2_Footprints:ESHF-105-01-L-D-SM -> SBV2_Footprints:SHF-105-01-L-D-SM
