File: eth.sch (KiCad schematic (older format))
At the start: 17 parts, among them P18 RJ45-HR911105A, U13 KSZ8081RNA, X2 25MHz

Commit message: Todo list changes: - series termination for ethernet - wired the three expansion ports - tied EN pins on drivers to gnd - added diode to 5V regulator supply - removed central via from ethernet PHY
Parts:
- added R107, R108, R109: 33R, Resistor_SMD:R_0402_1005Metric, symbol Smoothie2Standard-rescue:R
- C82, C83, C84, C85, C86, C87, C88, C89: symbol C -> Smoothie2Standard-rescue:C
- C90, C91: symbol C_Small -> Smoothie2Standard-rescue:C_Small
- L11: symbol INDUCTOR_SMALL -> Smoothie2Standard-rescue:INDUCTOR_SMALL
- P18: symbol RJ45-HR911105A -> rj45-hr911105a:RJ45-HR911105A
- R100, R98, R99: symbol R -> Smoothie2Standard-rescue:R
- U13: symbol KSZ8081RNA -> ksz8081rna:KSZ8081RNA
- X2: symbol CRYSTAL_SMD -> Smoothie2Standard-rescue:CRYSTAL_SMD
Connections:
- wire segments 79 -> 98
Changed lines of the file:
@@
-EESchema Schematic File Version 2
-LIBS:Smoothie2Standard-rescue
-LIBS:power
-LIBS:device
-LIBS:transistors
-LIBS:conn
-LIBS:linear
-LIBS:regul
-LIBS:74xx
-LIBS:cmos4000
-LIBS:adc-dac
-LIBS:memory
-LIBS:xilinx
-LIBS:microcontrollers
-LIBS:dsp
-LIBS:microchip
-LIBS:analog_switches
-LIBS:motorola
-LIBS:texas
-LIBS:intel
-LIBS:audio
-LIBS:interface
-LIBS:digital-audio
-LIBS:philips
-LIBS:display
-LIBS:cypress
-LIBS:siliconi
-LIBS:opto
-LIBS:atmel
-LIBS:contrib
-LIBS:valves
-LIBS:a4982
-LIBS:ap2511
-LIBS:ksz8081rna
-LIBS:lm1117
-LIBS:lpc43xxfet256
-LIBS:microsd
-LIBS:q_nmos_sssgd
-LIBS:r78e
-LIBS:spi_flash
-LIBS:a8498
-LIBS:s29glxxxs
-LIBS:tmc2660
-LIBS:rj45-hr911105a
-LIBS:tc4427a
-LIBS:Smoothie2Standard-cache
-EELAYER 25 0
+EESchema Schematic File Version 4
+EELAYER 30 0
 EELAYER END
 $Descr A4 11693 8268
@@
 $EndDescr
 $Comp
-L KSZ8081RNA U13
+L ksz8081rna:KSZ8081RNA U13
 U 1 1 59AD77E2
 P 4000 3300
@@
 $EndComp
 $Comp
-L RJ45-HR911105A P18
+L rj45-hr911105a:RJ45-HR911105A P18
 U 1 1 59AD7817
 P 9300 2600
@@
 $EndComp
 $Comp
-L CRYSTAL_SMD X2
+L Smoothie2Standard-rescue:CRYSTAL_SMD X2
 U 1 1 59BE2598
 P 1700 4600
@@
 XI
 $Comp
-L R R98
+L Smoothie2Standard-rescue:R R98
 U 1 1 59BE26E8
 P 2550 4700
@@
 GND
 $Comp
-L INDUCTOR_SMALL L11
+L Smoothie2Standard-rescue:INDUCTOR_SMALL L11
 U 1 1 59BE28DB
 P 1950 2300
@@
 3.3V
 $Comp
-L R R99
+L Smoothie2Standard-rescue:R R99
 U 1 1 59BE3011
 P 7350 2900
@@
 $EndComp
 $Comp
-L R R100
+L Smoothie2Standard-rescue:R R100
 U 1 1 59BE305F
 P 7350 3100
@@
 RXC
 $Comp
-L C C88
+L Smoothie2Standard-rescue:C C88
 U 1 1 59BE355C
 P 7700 3350
@@
 $EndComp
 $Comp
-L C C89
+L Smoothie2Standard-rescue:C C89
 U 1 1 59BE35CD
 P 8000 3350
@@
 	2300 4500 2300 4600
 Wire Wire Line
-	2300 4600 1900 4600
+	2300 4600 2100 4600
 Wire Wire Line
 	1500 4600 1300 4600
 Wire Wire Line
-	1300 4400 1300 4700
+	1300 4400 1300 4600
 Wire Wire Line
 	1300 4400 2800 4400
@@
 	2300 4700 2300 5000
 Wire Wire Line
-	2300 5000 1300 5000
-Wire Wire Line
-	1700 4700 1700 5100
+	2300 5000 2100 5000
+Wire Wire Line
+	1700 4700 1700 5000
 Connection ~ 1700 5000
 Wire Wire Line
 	2300 4200 2800 4200
 Wire Wire Line
-	2700 2700 2700 2850
+	2700 2700 2700 2800
 Wire Wire Line
 	2700 2800 2800 2800
@@
 Connection ~ 2700 2800
 Wire Wire Line
-	2200 2300 2800 2300
+	2200 2300 2300 2300
 Wire Wire Line
 	2300 1900 2300 2300
@@
 	2700 2100 2800 2100
 Wire Wire Line
-	1600 1900 1600 2500
+	1600 1900 1600 2300
 Wire Wire Line
 	1600 2300 1700 2300
@@
 	2300 3100 2800 3100
 Wire Wire Line
-	2300 3200 2800 3200
-Wire Wire Line
-	2300 3300 2800 3300
-Wire Wire Line
-	2300 3400 2800 3400
+	2300 3200 2500 3200
+Wire Wire Line
+	2300 3300 2500 3300
+Wire Wire Line
+	2300 3400 2500 3400
 Wire Wire Line
 	2300 3500 2800 3500
@@
 	10000 3000 9900 3000
 Wire Wire Line
-	8100 1900 8100 3000
+	8100 1900 8100 2800
 Wire Wire Line
 	8100 2800 8200 2800
@@
 	7700 3500 7700 3600
 Wire Wire Line
-	7700 3600 8150 3600
-Wire Wire Line
-	8000 3500 8000 3700
+	7700 3600 8000 3600
+Wire Wire Line
+	8000 3500 8000 3600
 Connection ~ 8000 3600
 Text GLabel 8000 3700 0    60   Input ~ 0
 GND
 $Comp
-L C C83
+L Smoothie2Standard-rescue:C C83
 U 1 1 59BE3DF9
 P 2000 1250
@@
 $EndComp
 $Comp
-L C C82
+L Smoothie2Standard-rescue:C C82
 U 1 1 59BE3E8D
 P 1700 1250
@@
 $EndComp
 $Comp
-L C C84
+L Smoothie2Standard-rescue:C C84
 U 1 1 59BE3EE9
 P 2300 1250
@@
 $EndComp
 $Comp
-L C C85
+L Smoothie2Standard-rescue:C C85
 U 1 1 59BE3F3B
 P 2600 1250
@@
 $EndComp
 $Comp
-L C C86
+L Smoothie2Standard-rescue:C C86
 U 1 1 59BE3F96
 P 2900 1250
@@
 $EndComp
 $Comp
-L C C87
+L Smoothie2Standard-rescue:C C87
 U 1 1 59BE3FE8
 P 3200 1250
@@
 	1700 1400 1700 1500
 Wire Wire Line
-	1700 1500 3200 1500
+	1700 1500 2000 1500
 Wire Wire Line
 	2000 1500 2000 1400
@@
 Connection ~ 2600 1500
 Wire Wire Line
-	3200 1400 3200 1600
+	3200 1400 3200 1500
 Connection ~ 2900 1500
 Connection ~ 3200 1500
@@
 GND
 Wire Wire Line
-	1700 800  1700 1100
+	1700 800  1700 1000
 Wire Wire Line
 	1700 1000 2000 1000
@@
 	2000 1000 2000 1100
 Wire Wire Line
-	2300 800  2300 1100
+	2300 800  2300 1000
 Wire Wire Line
 	2300 1000 2600 1000
@@
 	2600 1000 2600 1100
 Wire Wire Line
-	2900 800  2900 1100
+	2900 800  2900 1000
 Wire Wire Line
 	2900 1000 3200 1000
@@
 3.3VE
 $Comp
-L PWR_FLAG #FLG011
+L power:PWR_FLAG #FLG011
 U 1 1 59EE950F
 P 2200 2300
@@
 $EndComp
 $Comp
-L C_Small C90
+L Smoothie2Standard-rescue:C_Small C90
 U 1 1 5A44FBD2
 P 1300 4800
@@
 $EndComp
 $Comp
-L C_Small C91
+L Smoothie2Standard-rescue:C_Small C91
 U 1 1 5A44FC8D
 P 2100 4800
@@
 Wire Wire Line
 	8150 2700 8200 2700
+Wire Wire Line
+	1700 5000 1300 5000
+Wire Wire Line
+	1700 5000 1700 5100
+Wire Wire Line
+	2700 2800 2700 2850
+Wire Wire Line
+	2300 2300 2800 2300
+Wire Wire Line
+	1600 2300 1600 2500
+Wire Wire Line
+	8100 2800 8100 3000
+Wire Wire Line
+	8000 3600 8150 3600
+Wire Wire Line
+	8000 3600 8000 3700
+Wire Wire Line
+	2000 1500 2300 1500
+Wire Wire Line
+	2300 1500 2600 1500
+Wire Wire Line
+	2600 1500 2900 1500
+Wire Wire Line
+	2900 1500 3200 1500
+Wire Wire Line
+	3200 1500 3200 1600
+Wire Wire Line
+	1700 1000 1700 1100
+Wire Wire Line
+	2300 1000 2300 1100
+Wire Wire Line
+	2900 1000 2900 1100
+Wire Wire Line
+	1300 4600 1300 4700
+Wire Wire Line
+	2100 4600 1900 4600
+Wire Wire Line
+	2100 5000 1700 5000
+$Comp
+L Smoothie2Standard-rescue:R R107
+U 1 1 6069FA98
+P 2650 3200
+F 0 "R107" V 2730 3200 50  0000 C CNN
+F 1 "33R" V 2650 3200 50  0000 C CNN
+F 2 "Resistor_SMD:R_0402_1005Metric" V 2580 3200 50  0001 C CNN
+F 3 "" H 2650 3200 50  0000 C CNN
+	1    2650 3200
+	0    -1   -1   0
+$EndComp
+$Comp
+L Smoothie2Standard-rescue:R R108
+U 1 1 606A34B5
+P 2650 3300
+F 0 "R108" V 2730 3300 50  0000 C CNN
+F 1 "33R" V 2650 3300 50  0000 C CNN
+F 2 "Resistor_SMD:R_0402_1005Metric" V 2580 3300 50  0001 C CNN
+F 3 "" H 2650 3300 50  0000 C CNN
+	1    2650 3300
+	0    -1   -1   0
+$EndComp
+$Comp
+L Smoothie2Standard-rescue:R R109
+U 1 1 606A693D
+P 2650 3400
+F 0 "R109" V 2730 3400 50  0000 C CNN
+F 1 "33R" V 2650 3400 50  0000 C CNN
+F 2 "Resistor_SMD:R_0402_1005Metric" V 2580 3400 50  0001 C CNN
+F 3 "" H 2650 3400 50  0000 C CNN
+	1    2650 3400
+	0    -1   -1   0
+$EndComp
 $EndSCHEMATC
