File: driver.sch (KiCad schematic (older format))
At the start: 20 parts, among them Q1 Si4542DY, Q2 Si4542DY, Q3 Si4542DY, Q4 Si4542DY, U1 TMC2590

Commit message: Fix flipped motor MOSFETS. Add reverse current block and current limit to 5V DC/DC supply. Add pullups to SD and card detect.
Other:
- moved on the sheet: Q13A, Q13B, Q14A, Q14B, Q15A, Q15B, Q16A, Q16B
Changed lines of the file:
@@
 L Transistor_FET:Si4542DY Q1
 U 1 1 60B4B35F
-P 5100 2500
+P 5100 3050
 AR Path="/60B406B9/60B4B35F" Ref="Q1"  Part="1"
 AR Path="/60CED0E3/60B4B35F" Ref="Q5"  Part="2"
@@
 AR Path="/60FEEB1A/60B4B35F" Ref="Q9"  Part="1"
 AR Path="/60FF2256/60B4B35F" Ref="Q13"  Part="1"
-F 0 "Q13" H 5305 2546 50  0000 L CNN
-F 1 "Si4542DY" H 5305 2455 50  0000 L CNN
-F 2 "Package_SO:SOIC-8_3.9x4.9mm_P1.27mm" H 5300 2425 50  0001 L CNN
-F 3 "https://www.onsemi.com/pub/Collateral/SI4542DY-D.PDF" H 5200 2500 50  0001 L CNN
-	1    5100 2500
-	1    0    0    1
+F 0 "Q13" H 5305 3096 50  0000 L CNN
+F 1 "Si4542DY" H 5305 3005 50  0000 L CNN
+F 2 "Package_SO:SOIC-8_3.9x4.9mm_P1.27mm" H 5300 2975 50  0001 L CNN
+F 3 "https://www.onsemi.com/pub/Collateral/SI4542DY-D.PDF" H 5200 3050 50  0001 L CNN
+	1    5100 3050
+	1    0    0    -1
 $EndComp
 $Comp
 L Transistor_FET:Si4542DY Q1
 U 2 1 60C7E19D
-P 5100 3050
+P 5100 2500
 AR Path="/60B406B9/60C7E19D" Ref="Q1"  Part="2"
 AR Path="/60CED0E3/60C7E19D" Ref="Q5"  Part="1"
@@
 AR Path="/60FEEB1A/60C7E19D" Ref="Q9"  Part="2"
 AR Path="/60FF2256/60C7E19D" Ref="Q13"  Part="2"
-F 0 "Q13" H 5305 3004 50  0000 L CNN
-F 1 "Si4542DY" H 5305 3095 50  0000 L CNN
-F 2 "Package_SO:SOIC-8_3.9x4.9mm_P1.27mm" H 5300 2975 50  0001 L CNN
-F 3 "https://www.onsemi.com/pub/Collateral/SI4542DY-D.PDF" H 5200 3050 50  0001 L CNN
-	2    5100 3050
-	1    0    0    -1
+F 0 "Q13" H 5305 2454 50  0000 L CNN
+F 1 "Si4542DY" H 5305 2545 50  0000 L CNN
+F 2 "Package_SO:SOIC-8_3.9x4.9mm_P1.27mm" H 5300 2425 50  0001 L CNN
+F 3 "https://www.onsemi.com/pub/Collateral/SI4542DY-D.PDF" H 5200 2500 50  0001 L CNN
+	2    5100 2500
+	1    0    0    1
 $EndComp
 Wire Wire Line
@@
 L Transistor_FET:Si4542DY Q3
 U 1 1 60C7E19E
-P 5850 2650
+P 5850 3150
 AR Path="/60B406B9/60C7E19E" Ref="Q3"  Part="1"
 AR Path="/60CED0E3/60C7E19E" Ref="Q7"  Part="2"
@@
 AR Path="/60FEEB1A/60C7E19E" Ref="Q11"  Part="1"
 AR Path="/60FF2256/60C7E19E" Ref="Q15"  Part="1"
-F 0 "Q15" H 6055 2696 50  0000 L CNN
-F 1 "Si4542DY" H 6055 2605 50  0000 L CNN
-F 2 "Package_SO:SOIC-8_3.9x4.9mm_P1.27mm" H 6050 2575 50  0001 L CNN
-F 3 "https://www.onsemi.com/pub/Collateral/SI4542DY-D.PDF" H 5950 2650 50  0001 L CNN
-	1    5850 2650
-	1    0    0    1
+F 0 "Q15" H 6055 3196 50  0000 L CNN
+F 1 "Si4542DY" H 6055 3105 50  0000 L CNN
+F 2 "Package_SO:SOIC-8_3.9x4.9mm_P1.27mm" H 6050 3075 50  0001 L CNN
+F 3 "https://www.onsemi.com/pub/Collateral/SI4542DY-D.PDF" H 5950 3150 50  0001 L CNN
+	1    5850 3150
+	1    0    0    -1
 $EndComp
 $Comp
 L Transistor_FET:Si4542DY Q3
 U 2 1 60C7E19F
-P 5850 3150
+P 5850 2650
 AR Path="/60B406B9/60C7E19F" Ref="Q3"  Part="2"
 AR Path="/60CED0E3/60C7E19F" Ref="Q7"  Part="1"
@@
 AR Path="/60FEEB1A/60C7E19F" Ref="Q11"  Part="2"
 AR Path="/60FF2256/60C7E19F" Ref="Q15"  Part="2"
-F 0 "Q15" H 6055 3104 50  0000 L CNN
-F 1 "Si4542DY" H 6055 3195 50  0000 L CNN
-F 2 "Package_SO:SOIC-8_3.9x4.9mm_P1.27mm" H 6050 3075 50  0001 L CNN
-F 3 "https://www.onsemi.com/pub/Collateral/SI4542DY-D.PDF" H 5950 3150 50  0001 L CNN
-	2    5850 3150
-	1    0    0    -1
+F 0 "Q15" H 6055 2604 50  0000 L CNN
+F 1 "Si4542DY" H 6055 2695 50  0000 L CNN
+F 2 "Package_SO:SOIC-8_3.9x4.9mm_P1.27mm" H 6050 2575 50  0001 L CNN
+F 3 "https://www.onsemi.com/pub/Collateral/SI4542DY-D.PDF" H 5950 2650 50  0001 L CNN
+	2    5850 2650
+	1    0    0    1
 $EndComp
 Wire Wire Line
@@
 L Transistor_FET:Si4542DY Q2
 U 1 1 60C7E1A3
-P 5100 3800
+P 5100 4350
 AR Path="/60B406B9/60C7E1A3" Ref="Q2"  Part="1"
 AR Path="/60CED0E3/60C7E1A3" Ref="Q6"  Part="2"
@@
 AR Path="/60FEEB1A/60C7E1A3" Ref="Q10"  Part="1"
 AR Path="/60FF2256/60C7E1A3" Ref="Q14"  Part="1"
-F 0 "Q14" H 5305 3846 50  0000 L CNN
-F 1 "Si4542DY" H 5305 3755 50  0000 L CNN
-F 2 "Package_SO:SOIC-8_3.9x4.9mm_P1.27mm" H 5300 3725 50  0001 L CNN
-F 3 "https://www.onsemi.com/pub/Collateral/SI4542DY-D.PDF" H 5200 3800 50  0001 L CNN
-	1    5100 3800
-	1    0    0    1
+F 0 "Q14" H 5305 4396 50  0000 L CNN
+F 1 "Si4542DY" H 5305 4305 50  0000 L CNN
+F 2 "Package_SO:SOIC-8_3.9x4.9mm_P1.27mm" H 5300 4275 50  0001 L CNN
+F 3 "https://www.onsemi.com/pub/Collateral/SI4542DY-D.PDF" H 5200 4350 50  0001 L CNN
+	1    5100 4350
+	1    0    0    -1
 $EndComp
 $Comp
 L Transistor_FET:Si4542DY Q2
 U 2 1 60C7E1A4
-P 5100 4350
+P 5100 3800
 AR Path="/60B406B9/60C7E1A4" Ref="Q2"  Part="2"
 AR Path="/60CED0E3/60C7E1A4" Ref="Q6"  Part="1"
@@
 AR Path="/60FEEB1A/60C7E1A4" Ref="Q10"  Part="2"
 AR Path="/60FF2256/60C7E1A4" Ref="Q14"  Part="2"
-F 0 "Q14" H 5305 4304 50  0000 L CNN
-F 1 "Si4542DY" H 5305 4395 50  0000 L CNN
-F 2 "Package_SO:SOIC-8_3.9x4.9mm_P1.27mm" H 5300 4275 50  0001 L CNN
-F 3 "https://www.onsemi.com/pub/Collateral/SI4542DY-D.PDF" H 5200 4350 50  0001 L CNN
-	2    5100 4350
-	1    0    0    -1
+F 0 "Q14" H 5305 3754 50  0000 L CNN
+F 1 "Si4542DY" H 5305 3845 50  0000 L CNN
+F 2 "Package_SO:SOIC-8_3.9x4.9mm_P1.27mm" H 5300 3725 50  0001 L CNN
+F 3 "https://www.onsemi.com/pub/Collateral/SI4542DY-D.PDF" H 5200 3800 50  0001 L CNN
+	2    5100 3800
+	1    0    0    1
 $EndComp
 Wire Wire Line
@@
 L Transistor_FET:Si4542DY Q4
 U 1 1 60C7E1A5
-P 5850 3950
+P 5850 4450
 AR Path="/60B406B9/60C7E1A5" Ref="Q4"  Part="1"
 AR Path="/60CED0E3/60C7E1A5" Ref="Q8"  Part="2"
@@
 AR Path="/60FEEB1A/60C7E1A5" Ref="Q12"  Part="1"
 AR Path="/60FF2256/60C7E1A5" Ref="Q16"  Part="1"
-F 0 "Q16" H 6055 3996 50  0000 L CNN
-F 1 "Si4542DY" H 6055 3905 50  0000 L CNN
-F 2 "Package_SO:SOIC-8_3.9x4.9mm_P1.27mm" H 6050 3875 50  0001 L CNN
-F 3 "https://www.onsemi.com/pub/Collateral/SI4542DY-D.PDF" H 5950 3950 50  0001 L CNN
-	1    5850 3950
-	1    0    0    1
+F 0 "Q16" H 6055 4496 50  0000 L CNN
+F 1 "Si4542DY" H 6055 4405 50  0000 L CNN
+F 2 "Package_SO:SOIC-8_3.9x4.9mm_P1.27mm" H 6050 4375 50  0001 L CNN
+F 3 "https://www.onsemi.com/pub/Collateral/SI4542DY-D.PDF" H 5950 4450 50  0001 L CNN
+	1    5850 4450
+	1    0    0    -1
 $EndComp
 $Comp
 L Transistor_FET:Si4542DY Q4
 U 2 1 60C7E1A6
-P 5850 4450
+P 5850 3950
 AR Path="/60B406B9/60C7E1A6" Ref="Q4"  Part="2"
 AR Path="/60CED0E3/60C7E1A6" Ref="Q8"  Part="1"
@@
 AR Path="/60FEEB1A/60C7E1A6" Ref="Q12"  Part="2"
 AR Path="/60FF2256/60C7E1A6" Ref="Q16"  Part="2"
-F 0 "Q16" H 6055 4404 50  0000 L CNN
-F 1 "Si4542DY" H 6055 4495 50  0000 L CNN
-F 2 "Package_SO:SOIC-8_3.9x4.9mm_P1.27mm" H 6050 4375 50  0001 L CNN
-F 3 "https://www.onsemi.com/pub/Collateral/SI4542DY-D.PDF" H 5950 4450 50  0001 L CNN
-	2    5850 4450
-	1    0    0    -1
-$EndComp
-Wire Wire Line
+F 0 "Q16" H 6055 3904 50  0000 L CNN
+F 1 "Si4542DY" H 6055 3995 50  0000 L CNN
+F 2 "Package_SO:SOIC-8_3.9x4.9mm_P1.27mm" H 6050 3875 50  0001 L CNN
+F 3 "https://www.onsemi.com/pub/Collateral/SI4542DY-D.PDF" H 5950 3950 50  0001 L CNN
+	2    5850 3950
+	1    0    0    1
+$EndComp
+Wire Wire Line

Commit message: Move board thermistor, move LED resistors, add diode to probe input, NC header on probe input, change pullup on probe input, change value of enable resistor for fet driver, add ideal diode to schmatic, add fiducials to board, swap T1 and T4 opamp output
Parts:
- U1: symbol smoothieparts:TMC2590 -> smoothiev2-prime-rescue:TMC2590-smoothieparts
Changed lines of the file:
@@
 $Descr A4 11693 8268
 encoding utf-8
-Sheet 3 10
+Sheet 3 13
 Title ""
 Date ""
@@
 $EndDescr
 $Comp
-L smoothieparts:TMC2590 U1
+L smoothiev2-prime-rescue:TMC2590-smoothieparts U1
 U 1 1 60B43DE0
 P 3400 3450

Commit message: Adapt 2590 board layout to ideal diodes and dual power input connector
Parts:
- U1: symbol smoothiev2-prime-rescue:TMC2590-smoothieparts -> smoothiev2-prime-rescue:TMC2590-smoothieparts-smoothiev2-prime-rescue
Changed lines of the file:
@@
 $Descr A4 11693 8268
 encoding utf-8
-Sheet 3 13
+Sheet 5 13
 Title ""
 Date ""
@@
 $EndDescr
 $Comp
-L smoothiev2-prime-rescue:TMC2590-smoothieparts U1
+L smoothiev2-prime-rescue:TMC2590-smoothieparts-smoothiev2-prime-rescue U1
 U 1 1 60B43DE0
 P 3400 3450
@@
 AR Path="/60FEEB1A/60B43DE0" Ref="U6"  Part="1"
 AR Path="/60FF2256/60B43DE0" Ref="U7"  Part="1"
-F 0 "U7" H 3450 1661 50  0000 C CNN
+AR Path="/60B43DE0" Ref="U7"  Part="1"
+F 0 "U6" H 3450 1661 50  0000 C CNN
 F 1 "TMC2590" H 3450 1570 50  0000 C CNN
 F 2 "smoothieparts:TMC2590-TA-T" H 3100 2900 50  0001 C CNN
@@
 AR Path="/60FEEB1A/60B469D4" Ref="C31"  Part="1"
 AR Path="/60FF2256/60B469D4" Ref="C40"  Part="1"
-F 0 "C40" H 4415 2196 50  0000 L CNN
+F 0 "C31" H 4415 2196 50  0000 L CNN
 F 1 "1u" H 4415 2105 50  0000 L CNN
 F 2 "Capacitor_SMD:C_0402_1005Metric" H 4338 2000 50  0001 C CNN
@@
 AR Path="/60FEEB1A/60C7E19A" Ref="C29"  Part="1"
 AR Path="/60FF2256/60C7E19A" Ref="C38"  Part="1"
-F 0 "C38" H 3665 1796 50  0000 L CNN
+F 0 "C29" H 3665 1796 50  0000 L CNN
 F 1 "10u" H 3665 1705 50  0000 L CNN
 F 2 "Capacitor_SMD:C_0603_1608Metric" H 3588 1600 50  0001 C CNN
@@
 AR Path="/60FEEB1A/60B4812A" Ref="C28"  Part="1"
 AR Path="/60FF2256/60B4812A" Ref="C37"  Part="1"
-F 0 "C37" H 3265 1796 50  0000 L CNN
+F 0 "C28" H 3265 1796 50  0000 L CNN
 F 1 "1u" H 3265 1705 50  0000 L CNN
 F 2 "Capacitor_SMD:C_0402_1005Metric" H 3188 1600 50  0001 C CNN
@@
 AR Path="/60FEEB1A/60B4B35F" Ref="Q9"  Part="1"
 AR Path="/60FF2256/60B4B35F" Ref="Q13"  Part="1"
-F 0 "Q13" H 5305 3096 50  0000 L CNN
+F 0 "Q9" H 5305 3096 50  0000 L CNN
 F 1 "Si4542DY" H 5305 3005 50  0000 L CNN
 F 2 "Package_SO:SOIC-8_3.9x4.9mm_P1.27mm" H 5300 2975 50  0001 L CNN
@@
 AR Path="/60FEEB1A/60C7E19D" Ref="Q9"  Part="2"
 AR Path="/60FF2256/60C7E19D" Ref="Q13"  Part="2"
-F 0 "Q13" H 5305 2454 50  0000 L CNN
+F 0 "Q9" H 5305 2454 50  0000 L CNN
 F 1 "Si4542DY" H 5305 2545 50  0000 L CNN
 F 2 "Package_SO:SOIC-8_3.9x4.9mm_P1.27mm" H 5300 2425 50  0001 L CNN
@@
 AR Path="/60FEEB1A/60C7E19E" Ref="Q11"  Part="1"
 AR Path="/60FF2256/60C7E19E" Ref="Q15"  Part="1"
-F 0 "Q15" H 6055 3196 50  0000 L CNN
+F 0 "Q11" H 6055 3196 50  0000 L CNN
 F 1 "Si4542DY" H 6055 3105 50  0000 L CNN
 F 2 "Package_SO:SOIC-8_3.9x4.9mm_P1.27mm" H 6050 3075 50  0001 L CNN
@@
 AR Path="/60FEEB1A/60C7E19F" Ref="Q11"  Part="2"
 AR Path="/60FF2256/60C7E19F" Ref="Q15"  Part="2"
-F 0 "Q15" H 6055 2604 50  0000 L CNN
+F 0 "Q11" H 6055 2604 50  0000 L CNN
 F 1 "Si4542DY" H 6055 2695 50  0000 L CNN
 F 2 "Package_SO:SOIC-8_3.9x4.9mm_P1.27mm" H 6050 2575 50  0001 L CNN
@@
 AR Path="/60FEEB1A/60B5CCDD" Ref="R25"  Part="1"
 AR Path="/60FF2256/60B5CCDD" Ref="R29"  Part="1"
-F 0 "R29" V 4793 3600 50  0000 C CNN
+F 0 "R25" V 4793 3600 50  0000 C CNN
 F 1 "R" V 4884 3600 50  0000 C CNN
 F 2 "Resistor_SMD:R_2512_6332Metric" V 4930 3600 50  0001 C CNN
@@
 AR Path="/60FEEB1A/60C7E1A1" Ref="R23"  Part="1"
 AR Path="/60FF2256/60C7E1A1" Ref="R27"  Part="1"
-F 0 "R27" V 4443 3450 50  0000 C CNN
+F 0 "R23" V 4443 3450 50  0000 C CNN
 F 1 "47R" V 4534 3450 50  0000 C CNN
 F 2 "Resistor_SMD:R_0402_1005Metric" V 4580 3450 50  0001 C CNN
@@
 AR Path="/60FEEB1A/60C7E1A2" Ref="C30"  Part="1"
 AR Path="/60FF2256/60C7E1A2" Ref="C39"  Part="1"
-F 0 "C39" H 4065 1846 50  0000 L CNN
+F 0 "C30" H 4065 1846 50  0000 L CNN
 F 1 "100n" H 4065 1755 50  0000 L CNN
 F 2 "Capacitor_SMD:C_0402_1005Metric" H 3988 1650 50  0001 C CNN
@@
 AR Path="/60FEEB1A/60C7E1A3" Ref="Q10"  Part="1"
 AR Path="/60FF2256/60C7E1A3" Ref="Q14"  Part="1"
-F 0 "Q14" H 5305 4396 50  0000 L CNN
+F 0 "Q10" H 5305 4396 50  0000 L CNN
 F 1 "Si4542DY" H 5305 4305 50  0000 L CNN
 F 2 "Package_SO:SOIC-8_3.9x4.9mm_P1.27mm" H 5300 4275 50  0001 L CNN
@@
 AR Path="/60FEEB1A/60C7E1A4" Ref="Q10"  Part="2"
 AR Path="/60FF2256/60C7E1A4" Ref="Q14"  Part="2"
-F 0 "Q14" H 5305 3754 50  0000 L CNN
+F 0 "Q10" H 5305 3754 50  0000 L CNN
 F 1 "Si4542DY" H 5305 3845 50  0000 L CNN
 F 2 "Package_SO:SOIC-8_3.9x4.9mm_P1.27mm" H 5300 3725 50  0001 L CNN
@@
 AR Path="/60FEEB1A/60C7E1A5" Ref="Q12"  Part="1"
 AR Path="/60FF2256/60C7E1A5" Ref="Q16"  Part="1"
-F 0 "Q16" H 6055 4496 50  0000 L CNN
+F 0 "Q12" H 6055 4496 50  0000 L CNN
 F 1 "Si4542DY" H 6055 4405 50  0000 L CNN
 F 2 "Package_SO:SOIC-8_3.9x4.9mm_P1.27mm" H 6050 4375 50  0001 L CNN
@@
 AR Path="/60FEEB1A/60C7E1A6" Ref="Q12"  Part="2"
 AR Path="/60FF2256/60C7E1A6" Ref="Q16"  Part="2"
-F 0 "Q16" H 6055 3904 50  0000 L CNN
+F 0 "Q12" H 6055 3904 50  0000 L CNN
 F 1 "Si4542DY" H 6055 3995 50  0000 L CNN
 F 2 "Package_SO:SOIC-8_3.9x4.9mm_P1.27mm" H 6050 3875 50  0001 L CNN
@@
 AR Path="/60FEEB1A/60C7E1A7" Ref="R26"  Part="1"
 AR Path="/60FF2256/60C7E1A7" Ref="R30"  Part="1"
-F 0 "R30" V 4793 4900 50  0000 C CNN
+F 0 "R26" V 4793 4900 50  0000 C CNN
 F 1 "R" V 4884 4900 50  0000 C CNN
 F 2 "Resistor_SMD:R_2512_6332Metric" V 4930 4900 50  0001 C CNN
@@
 AR Path="/60FEEB1A/60C7E1A8" Ref="R24"  Part="1"
 AR Path="/60FF2256/60C7E1A8" Ref="R28"  Part="1"
-F 0 "R28" V 4443 4750 50  0000 C CNN
+F 0 "R24" V 4443 4750 50  0000 C CNN
 F 1 "47R" V 4534 4750 50  0000 C CNN
 F 2 "Resistor_SMD:R_0402_1005Metric" V 4580 4750 50  0001 C CNN
@@
 AR Path="/60FEEB1A/60C1AD6E" Ref="C33"  Part="1"
 AR Path="/60FF2256/60C1AD6E" Ref="C42"  Part="1"
-F 0 "C42" H 6915 2496 50  0000 L CNN
+F 0 "C33" H 6915 2496 50  0000 L CNN
 F 1 "10u" H 6915 2405 50  0000 L CNN
 F 2 "Capacitor_SMD:C_1206_3216Metric" H 6838 2300 50  0001 C CNN
@@
 AR Path="/60FEEB1A/60C7E1AA" Ref="C32"  Part="1"
 AR Path="/60FF2256/60C7E1AA" Ref="C41"  Part="1"
-F 0 "C41" H 6565 2496 50  0000 L CNN
+F 0 "C32" H 6565 2496 50  0000 L CNN
 F 1 "10u" H 6565 2405 50  0000 L CNN
 F 2 "Capacitor_SMD:C_1206_3216Metric" H 6488 2300 50  0001 C CNN
@@
 AR Path="/60FEEB1A/60C7E1AB" Ref="C34"  Part="1"
 AR Path="/60FF2256/60C7E1AB" Ref="C43"  Part="1"
-F 0 "C43" H 7265 2496 50  0000 L CNN
+F 0 "C34" H 7265 2496 50  0000 L CNN
 F 1 "10u" H 7265 2405 50  0000 L CNN
 F 2 "Capacitor_SMD:C_1206_3216Metric" H 7188 2300 50  0001 C CNN
@@
 AR Path="/60FEEB1A/60C7E1AC" Ref="C35"  Part="1"
 AR Path="/60FF2256/60C7E1AC" Ref="C44"  Part="1"
-F 0 "C44" H 7615 2496 50  0000 L CNN
+F 0 "C35" H 7615 2496 50  0000 L CNN
 F 1 "10u" H 7615 2405 50  0000 L CNN
 F 2 "Capacitor_SMD:C_1206_3216Metric" H 7538 2300 50  0001 C CNN
@@
 AR Path="/60FEEB1A/60C36F84" Ref="C36"  Part="1"
 AR Path="/60FF2256/60C36F84" Ref="C45"  Part="1"
-F 0 "C45" H 8018 2496 50  0000 L CNN
+F 0 "C36" H 8018 2496 50  0000 L CNN
 F 1 "CP" H 8018 2405 50  0000 L CNN
 F 2 "Capacitor_SMD:CP_Elec_8x11.9" H 7938 2300 50  0001 C CNN
@@
 AR Path="/60FEEB1A/60C4D4FD" Ref="NT6"  Part="1"
 AR Path="/60FF2256/60C4D4FD" Ref="NT8"  Part="1"
-F 0 "NT8" H 4750 5231 50  0000 C CNN
+F 0 "NT6" H 4750 5231 50  0000 C CNN
 F 1 "Net-Tie_2" H 4750 5140 50  0000 C CNN
 F 2 "smoothieparts:NetTie-2_SMD_Pad2.0mm" H 4750 5050 50  0001 C CNN
@@
 AR Path="/60FEEB1A/60C7E1AF" Ref="NT5"  Part="1"
 AR Path="/60FF2256/60C7E1AF" Ref="NT7"  Part="1"
-F 0 "NT7" H 4700 3881 50  0000 C CNN
+F 0 "NT5" H 4700 3881 50  0000 C CNN
 F 1 "Net-Tie_2" H 4700 3790 50  0000 C CNN
 F 2 "smoothieparts:NetTie-2_SMD_Pad2.0mm" H 4700 3700 50  0001 C CNN

Commit message: Fix JP7 footprint, fix silk, add traces to vfet header
Parts:
- U1: symbol smoothiev2-prime-rescue:TMC2590-smoothieparts-smoothiev2-prime-rescue -> smoothiev2-prime-rescue:TMC2590-smoothieparts-smoothiev2-prime-rescue-smoothiev2-prime-rescue
Changed lines of the file:
@@
 $EndDescr
 $Comp
-L smoothiev2-prime-rescue:TMC2590-smoothieparts-smoothiev2-prime-rescue U1
+L smoothiev2-prime-rescue:TMC2590-smoothieparts-smoothiev2-prime-rescue-smoothiev2-prime-rescue U1
 U 1 1 60B43DE0
 P 3400 3450
