File: smoothiev2-prime.sch (KiCad schematic (older format))
At the start: 144 parts, among them J1 USB_B, J10 Conn_01x02, J15 Conn_01x02, J2 USB_A, J3 Micro_SD_Card_Det, J30 Conn_01x03_Male, J41 Conn_ARM_JTAG_SWD_10, J42 Conn_01x02, J43 Conn_01x02, J5 Screw_Terminal_01x04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

Commit message: Move board thermistor, move LED resistors, add diode to probe input, NC header on probe input, change pullup on probe input, change value of enable resistor for fet driver, add ideal diode to schmatic, add fiducials to board, swap T1 and T4 opamp output
Parts:
- added FID1, FID2, FID3, FID4: Fiducial, Fiducials:Fiducial_0.75mm_Dia_1.5mm_Outer, symbol Mechanical:Fiducial
- U2: symbol smoothieparts:STM32H745XIHx -> smoothiev2-prime-rescue:STM32H745XIHx-smoothieparts
Changed lines of the file:
@@
 $Descr A3 11693 16535 portrait
 encoding utf-8
-Sheet 1 10
+Sheet 1 13
 Title ""
 Date ""
@@
 Connection ~ 5250 12750
 $Comp
-L smoothieparts:STM32H745XIHx U2
+L smoothiev2-prime-rescue:STM32H745XIHx-smoothieparts U2
 U 1 1 607B3889
 P 7550 7450
@@
 PROBE
 $Sheet
-S 5250 650  650  900
+S 5250 650  625  975
 U 631D7D17
 F0 "power" 50
@@
 F8 "3V3_LIM" I L 5250 1350 50
 F9 "VBAT" I L 5250 1450 50
+F10 "USB_PWR" I L 5250 1550 50
 $EndSheet
 $Comp
@@
 	1    0    0    -1
 $EndComp
+Text Label 5250 1550 2    50   ~ 0
+USB_PWR
+$Comp
+L Mechanical:Fiducial FID1
+U 1 1 63978589
+P 9150 14925
+F 0 "FID1" H 9235 14971 50  0000 L CNN
+F 1 "Fiducial" H 9235 14880 50  0000 L CNN
+F 2 "Fiducials:Fiducial_0.75mm_Dia_1.5mm_Outer" H 9150 14925 50  0001 C CNN
+F 3 "~" H 9150 14925 50  0001 C CNN
+	1    9150 14925
+	1    0    0    -1
+$EndComp
+$Comp
+L Mechanical:Fiducial FID2
+U 1 1 63978B07
+P 9150 15100
+F 0 "FID2" H 9235 15146 50  0000 L CNN
+F 1 "Fiducial" H 9235 15055 50  0000 L CNN
+F 2 "Fiducials:Fiducial_0.75mm_Dia_1.5mm_Outer" H 9150 15100 50  0001 C CNN
+F 3 "~" H 9150 15100 50  0001 C CNN
+	1    9150 15100
+	1    0    0    -1
+$EndComp
+$Comp
+L Mechanical:Fiducial FID3
+U 1 1 63978E0C
+P 9650 14925
+F 0 "FID3" H 9735 14971 50  0000 L CNN
+F 1 "Fiducial" H 9735 14880 50  0000 L CNN
+F 2 "Fiducials:Fiducial_0.75mm_Dia_1.5mm_Outer" H 9650 14925 50  0001 C CNN
+F 3 "~" H 9650 14925 50  0001 C CNN
+	1    9650 14925
+	1    0    0    -1
+$EndComp
+$Comp
+L Mechanical:Fiducial FID4
+U 1 1 63979453
+P 9650 15100
+F 0 "FID4" H 9735 15146 50  0000 L CNN
+F 1 "Fiducial" H 9735 15055 50  0000 L CNN
+F 2 "Fiducials:Fiducial_0.75mm_Dia_1.5mm_Outer" H 9650 15100 50  0001 C CNN
+F 3 "~" H 9650 15100 50  0001 C CNN
+	1    9650 15100
+	1    0    0    -1
+$EndComp

Commit message: Adapt 2590 board layout to ideal diodes and dual power input connector
Parts:
- U2: symbol smoothiev2-prime-rescue:STM32H745XIHx-smoothieparts -> smoothiev2-prime-rescue:STM32H745XIHx-smoothieparts-smoothiev2-prime-rescue
Connections:
- net labels added: 5V_PORTIN
Changed lines of the file:
@@
 Connection ~ 5250 12750
 $Comp
-L smoothiev2-prime-rescue:STM32H745XIHx-smoothieparts U2
+L smoothiev2-prime-rescue:STM32H745XIHx-smoothieparts-smoothiev2-prime-rescue U2
 U 1 1 607B3889
 P 7550 7450
@@
 Text Label 10450 5150 0    50   ~ 0
 PROBE
-$Sheet
-S 5250 650  625  975
-U 631D7D17
-F0 "power" 50
-F1 "power.sch" 50
-F2 "5VIN" I L 5250 750 50
-F3 "5VOUT" I L 5250 850 50
-F4 "VMOT" I L 5250 950 50
-F5 "VMOTSENSE" I L 5250 1050 50
-F6 "3V3_DCDC" I L 5250 1150 50
-F7 "5V_LIM" I L 5250 1250 50
-F8 "3V3_LIM" I L 5250 1350 50
-F9 "VBAT" I L 5250 1450 50
-F10 "USB_PWR" I L 5250 1550 50
-$EndSheet
 $Comp
 L Connector_Generic:Conn_01x02 J43
@@
 	1    0    0    -1
 $EndComp
-Text Label 7400 1250 0    50   ~ 0
-5V_IN
+Text Label 5250 850  2    50   ~ 0
+5V_PORTIN
 $Comp
 L power:GND #PWR034
@@
 Text Label 5250 950  2    50   ~ 0
 VMOT
-Text Label 5250 850  2    50   ~ 0
+Text Label 5850 750  0    50   ~ 0
 5V
 Text Label 5250 750  2    50   ~ 0
@@
 	1    0    0    -1
 $EndComp
-Text Label 5250 1550 2    50   ~ 0
-USB_PWR
 $Comp
 L Mechanical:Fiducial FID1
@@
 	1    0    0    -1
 $EndComp
+$Sheet
+S 5250 650  600  1000
+U 631D7D17
+F0 "power" 50
+F1 "power.sch" 50
+F2 "5VIN" I L 5250 750 50
+F3 "5VOUT" I R 5850 750 50
+F4 "VMOT" I L 5250 950 50
+F5 "VMOTSENSE" I L 5250 1050 50
+F6 "3V3_DCDC" I L 5250 1150 50
+F7 "5V_LIM" I L 5250 1250 50
+F8 "3V3_LIM" I L 5250 1350 50
+F9 "VBAT" I L 5250 1450 50
+F10 "5V_PORTIN" I L 5250 850 50
+$EndSheet
+Text Label 7400 1250 0    50   ~ 0
+5V_PORTIN
 $EndSCHEMATC

Commit message: Fix JP7 footprint, fix silk, add traces to vfet header
Parts:
- U2: symbol smoothiev2-prime-rescue:STM32H745XIHx-smoothieparts-smoothiev2-prime-rescue -> smoothiev2-prime-rescue:STM32H745XIHx-smoothieparts-smoothiev2-prime-rescue-smoothiev2-prime-rescue
Changed lines of the file:
@@
 Connection ~ 5250 12750
 $Comp
-L smoothiev2-prime-rescue:STM32H745XIHx-smoothieparts-smoothiev2-prime-rescue U2
+L smoothiev2-prime-rescue:STM32H745XIHx-smoothieparts-smoothiev2-prime-rescue-smoothiev2-prime-rescue U2
 U 1 1 607B3889
 P 7550 7450
