File: driver-2660.sch (KiCad schematic (older format))
At the start: 13 parts, among them U3 TMC2660

Commit message: Updated 2660 version to match 2590 mods.
Updated 2660 version to match 2590 mods.  Ideal diodes, move board thermistor, add extra fet connector, modify probe input.
Parts:
- U3: symbol smoothieparts:TMC2660 -> smoothiev2-prime-2660-rescue:TMC2660-smoothieparts
Changed lines of the file:
@@
 $EndDescr
 $Comp
-L smoothieparts:TMC2660 U3
+L smoothiev2-prime-2660-rescue:TMC2660-smoothieparts U3
 U 1 1 6201210C
 P 4100 3750
