File: ethernet.sch (KiCad schematic (older format))
At the start: 29 parts, among them J4 RJ45_Hanrun_HR911105A, U1 LAN8720A, U10 TPD4E1U06DCKR, Y1 Crystal_GND24

Commit message: Move board thermistor, move LED resistors, add diode to probe input, NC header on probe input, change pullup on probe input, change value of enable resistor for fet driver, add ideal diode to schmatic, add fiducials to board, swap T1 and T4 opamp output
Parts:
- J4: symbol smoothieparts:RJ45_Hanrun_HR911105A -> smoothiev2-prime-rescue:RJ45_Hanrun_HR911105A-smoothieparts
Changed lines of the file:
@@
 $Descr A4 11693 8268
 encoding utf-8
-Sheet 2 10
+Sheet 2 13
 Title ""
 Date ""
@@
 	6950 5350 7050 5350
 $Comp
-L smoothieparts:RJ45_Hanrun_HR911105A J4
+L smoothiev2-prime-rescue:RJ45_Hanrun_HR911105A-smoothieparts J4
 U 1 1 60DC8A27
 P 7450 4150

Commit message: Adapt 2590 board layout to ideal diodes and dual power input connector
Parts:
- J4: symbol smoothiev2-prime-rescue:RJ45_Hanrun_HR911105A-smoothieparts -> smoothiev2-prime-rescue:RJ45_Hanrun_HR911105A-smoothieparts-smoothiev2-prime-rescue
Changed lines of the file:
@@
 	6950 5350 7050 5350
 $Comp
-L smoothiev2-prime-rescue:RJ45_Hanrun_HR911105A-smoothieparts J4
+L smoothiev2-prime-rescue:RJ45_Hanrun_HR911105A-smoothieparts-smoothiev2-prime-rescue J4
 U 1 1 60DC8A27
 P 7450 4150
+AR Path="/60DC8A27" Ref="J4"  Part="1"
+AR Path="/60D8BE45/60DC8A27" Ref="J4"  Part="1"
 F 0 "J4" H 6920 4196 50  0000 R CNN
 F 1 "RJ45_Hanrun_HR911105A" H 6920 4105 50  0000 R CNN

Commit message: Updated 2660 version to match 2590 mods.
Updated 2660 version to match 2590 mods.  Ideal diodes, move board thermistor, add extra fet connector, modify probe input.
Parts:
- J4: symbol smoothiev2-prime-rescue:RJ45_Hanrun_HR911105A-smoothieparts-smoothiev2-prime-rescue -> smoothiev2-prime-2660-rescue:RJ45_Hanrun_HR911105A-smoothieparts-smoothiev2-prime-rescue-smoothiev2-prime-rescue
Changed lines of the file:
@@
 	6950 5350 7050 5350
 $Comp
-L smoothiev2-prime-rescue:RJ45_Hanrun_HR911105A-smoothieparts-smoothiev2-prime-rescue J4
+L smoothiev2-prime-2660-rescue:RJ45_Hanrun_HR911105A-smoothieparts-smoothiev2-prime-rescue-smoothiev2-prime-rescue J4
 U 1 1 60DC8A27
 P 7450 4150
