File: power.sch (KiCad schematic (older format))
At the start: 41 parts, among them U18 MT9700, U19 MT9700, U20 MT9700, U21 TPS5430DDA, U22 MT3410L, U23 AP22814AW5

Commit message: Add power monitor circuit to VMOT DC/DC, add disconnect jumper to 5V_IN USB.
Parts:
- removed C117: 22u, Capacitor_SMD:C_0805_2012Metric, symbol Device:C
- added R100: 21.5k, Resistor_SMD:R_0402_1005Metric, symbol Device:R
- added R99: 56k, Resistor_SMD:R_0402_1005Metric, symbol Device:R
- added U25: BD4722G, Package_TO_SOT_SMD:SOT-23-5, symbol smoothieparts:BD47XXG
Connections:
- net labels added: UVLO
- wire segments 69 -> 74
Other:
- note added: "VMOT UNDERVOLTAGE DETECT"
Changed lines of the file:
@@
 $Descr A4 11693 8268
 encoding utf-8
-Sheet 6 10
+Sheet 10 10
 Title ""
 Date ""
@@
 $EndComp
 Wire Wire Line
-	1750 3950 2400 3950
+	1750 3950 2150 3950
 Wire Wire Line
 	4500 2700 4750 2700
@@
 Text HLabel 7600 2700 1    50   Input ~ 0
 3V3_DCDC
-$Comp
-L Device:C C117
-U 1 1 63E25811
-P 3150 2850
-F 0 "C117" H 3265 2896 50  0000 L CNN
-F 1 "22u" H 3265 2805 50  0000 L CNN
-F 2 "Capacitor_SMD:C_0805_2012Metric" H 3188 2700 50  0001 C CNN
-F 3 "~" H 3150 2850 50  0001 C CNN
-	1    3150 2850
-	1    0    0    -1
-$EndComp
 Wire Wire Line
 	3150 2700 3400 2700
 Connection ~ 3400 2700
-Wire Wire Line
-	3150 3000 3400 3000
-Connection ~ 3400 3000
 Wire Wire Line
 	8000 2700 7600 2700
@@
 Wire Notes Line
 	2250 2150 2250 3600
-Wire Notes Line
-	750  2150 750  5100
 Wire Notes Line
 	7750 2150 7750 5100
@@
 	6550 3350 6550 3950
 Wire Wire Line
-	6550 4250 6250 4250
-Wire Wire Line
 	6050 4250 6050 3950
 Wire Wire Line
@@
 Wire Wire Line
 	6550 4450 6250 4450
-Wire Wire Line
-	6250 4450 6250 4250
-Connection ~ 6250 4250
-Wire Wire Line
-	6250 4250 6050 4250
 NoConn ~ 7350 4450
 $Comp
@@
 Wire Wire Line
 	5600 3950 5350 3950
+Wire Wire Line
+	6050 4250 6550 4250
+Text Label 6250 4450 2    50   ~ 0
+UVLO
+Text Label 3250 4350 2    50   ~ 0
+UVLO
+$Comp
+L smoothieparts:BD47XXG U25
+U 1 1 627CE557
+P 2550 5800
+F 0 "U25" H 2362 5871 50  0000 R CNN
+F 1 "BD4722G" H 2850 6150 50  0000 R CNN
+F 2 "Package_TO_SOT_SMD:SOT-23-5" H 2550 5800 50  0001 C CNN
+F 3 "" H 2550 5800 50  0001 C CNN
+	1    2550 5800
+	1    0    0    -1
+$EndComp
+Text Label 2850 5650 0    50   ~ 0
+UVLO
+$Comp
+L power:GND #PWR?
+U 1 1 627D26CD
+P 2450 6100
+AR Path="/627D26CD" Ref="#PWR?"  Part="1"
+AR Path="/631D7D17/627D26CD" Ref="#PWR076"  Part="1"
+F 0 "#PWR076" H 2450 5850 50  0001 C CNN
+F 1 "GND" H 2455 5927 50  0000 C CNN
+F 2 "" H 2450 6100 50  0001 C CNN
+F 3 "" H 2450 6100 50  0001 C CNN
+	1    2450 6100
+	1    0    0    -1
+$EndComp
+Wire Wire Line
+	2550 6100 2450 6100
+Connection ~ 2450 6100
+$Comp
+L Device:R R?
+U 1 1 627D5521
+P 2050 5450
+AR Path="/627D5521" Ref="R?"  Part="1"
+AR Path="/631D7D17/627D5521" Ref="R99"  Part="1"
+F 0 "R99" H 2120 5496 50  0000 L CNN
+F 1 "56k" H 2120 5405 50  0000 L CNN
+F 2 "Resistor_SMD:R_0402_1005Metric" V 1980 5450 50  0001 C CNN
+F 3 "~" H 2050 5450 50  0001 C CNN
+	1    2050 5450
+	0    1    1    0
+$EndComp
+$Comp
+L Device:R R?
+U 1 1 627D6BF2
+P 2200 5950
+AR Path="/627D6BF2" Ref="R?"  Part="1"
+AR Path="/631D7D17/627D6BF2" Ref="R100"  Part="1"
+F 0 "R100" H 2270 5996 50  0000 L CNN
+F 1 "21.5k" H 2270 5905 50  0000 L CNN
+F 2 "Resistor_SMD:R_0402_1005Metric" V 2130 5950 50  0001 C CNN
+F 3 "~" H 2200 5950 50  0001 C CNN
+	1    2200 5950
+	-1   0    0    1
+$EndComp
+Wire Wire Line
+	2450 5450 2200 5450
+Wire Wire Line
+	2200 5450 2200 5800
+Connection ~ 2200 5450
+Wire Wire Line
+	2450 6100 2200 6100
+Wire Wire Line
+	1900 5450 1900 4600
+Wire Wire Line
+	1900 4600 2150 4600
+Wire Wire Line
+	2150 4600 2150 3950
+Connection ~ 2150 3950
+Wire Wire Line
+	2150 3950 2400 3950
+Wire Notes Line
+	750  6700 4100 6700
+Wire Notes Line
+	4100 6700 4100 5100
+Wire Notes Line
+	750  2150 750  6700
+Text Notes 850  6550 0    100  ~ 0
+VMOT UNDERVOLTAGE DETECT
 $EndSCHEMATC

Commit message: Move board thermistor, move LED resistors, add diode to probe input, NC header on probe input, change pullup on probe input, change value of enable resistor for fet driver, add ideal diode to schmatic, add fiducials to board, swap T1 and T4 opamp output
Parts:
- added R103: 33k, Resistors_SMD:R_0402, symbol Device:R
- added R104: 7.1k, Resistors_SMD:R_0402, symbol Device:R
- U25: symbol smoothieparts:BD47XXG -> smoothiev2-prime-rescue:BD47XXG-smoothieparts
Connections:
- net labels added: 5v_REG, 5v_USB, USB_PWR
- wire segments 74 -> 76
Changed lines of the file:
@@
 $Descr A4 11693 8268
 encoding utf-8
-Sheet 10 10
+Sheet 10 13
 Title ""
 Date ""
@@
 Comment4 ""
 $EndDescr
-Text HLabel 3150 2700 0    50   Input ~ 0
+Text HLabel 3825 1675 0    50   Input ~ 0
 5VIN
 Text HLabel 1750 3950 0    50   Input ~ 0
@@
 Connection ~ 7600 2700
 Connection ~ 7900 3950
-Wire Wire Line
-	5450 2700 5450 3350
 Connection ~ 5750 2700
-Connection ~ 4750 2700
 Wire Notes Line
 	6450 3600 6450 5100
@@
 Wire Notes Line
 	750  5100 9800 5100
-Wire Notes Line
-	750  2150 9800 2150
 Text Notes 2650 3500 0    50   ~ 10
 Current limit in A = 6.8k/R. Set to 1.44A with R63=4.7k
@@
 	1    0    0    -1
 $EndComp
-Connection ~ 5150 2700
-Wire Wire Line
-	5150 2700 4750 2700
 $Comp
 L power:GND #PWR?
@@
 	5550 2700 5750 2700
 Wire Wire Line
-	5450 3350 6550 3350
-Wire Wire Line
-	6550 3950 7350 3950
-Wire Wire Line
 	5050 3950 5350 3950
-Wire Wire Line
-	7350 4250 7350 3950
-Connection ~ 7350 3950
-Wire Wire Line
-	7350 3950 7900 3950
-Wire Wire Line
-	6550 3350 6550 3950
 Wire Wire Line
 	6050 4250 6050 3950
@@
 UVLO
 $Comp
-L smoothieparts:BD47XXG U25
+L smoothiev2-prime-rescue:BD47XXG-smoothieparts U25
 U 1 1 627CE557
 P 2550 5800
+AR Path="/627CE557" Ref="U25"  Part="1"
+AR Path="/631D7D17/627CE557" Ref="U25"  Part="1"
 F 0 "U25" H 2362 5871 50  0000 R CNN
 F 1 "BD4722G" H 2850 6150 50  0000 R CNN
@@
 	1    0    0    -1
 $EndComp
-Text Label 2850 5650 0    50   ~ 0
+Text Label 3125 5650 0    50   ~ 0
 UVLO
 $Comp
@@
 	2450 6100 2200 6100
 Wire Wire Line
-	1900 5450 1900 4600
+	1900 5450 1900 5350
 Wire Wire Line
 	1900 4600 2150 4600
@@
 Text Notes 850  6550 0    100  ~ 0
 VMOT UNDERVOLTAGE DETECT
+$Comp
+L Device:R R?
+U 1 1 63875BD8
+P 2975 5800
+AR Path="/63875BD8" Ref="R?"  Part="1"
+AR Path="/631D7D17/63875BD8" Ref="R104"  Part="1"
+F 0 "R104" H 3045 5846 50  0000 L CNN
+F 1 "7.1k" H 3045 5755 50  0000 L CNN
+F 2 "Resistors_SMD:R_0402" V 2905 5800 50  0001 C CNN
+F 3 "~" H 2975 5800 50  0001 C CNN
+	1    2975 5800
+	1    0    0    -1
+$EndComp
+$Comp
+L Device:R R?
+U 1 1 63876832
+P 2975 5500
+AR Path="/63876832" Ref="R?"  Part="1"
+AR Path="/631D7D17/63876832" Ref="R103"  Part="1"
+F 0 "R103" H 3045 5546 50  0000 L CNN
+F 1 "33k" H 3045 5455 50  0000 L CNN
+F 2 "Resistors_SMD:R_0402" V 2905 5500 50  0001 C CNN
+F 3 "~" H 2975 5500 50  0001 C CNN
+	1    2975 5500
+	1    0    0    -1
+$EndComp
+Wire Wire Line
+	2975 5350 1900 5350
+Connection ~ 1900 5350
+Wire Wire Line
+	1900 5350 1900 4600
+Wire Wire Line
+	2975 5950 2975 6100
+Wire Wire Line
+	2975 6100 2550 6100
+Connection ~ 2550 6100
+Wire Wire Line
+	2850 5650 2975 5650
+Connection ~ 2975 5650
+Wire Wire Line
+	2975 5650 3125 5650
+Wire Notes Line
+	750  2150 9800 2150
+$Sheet
+S 3825 1625 525  200
+U 63881870
+F0 "IdealDiode" 50
+F1 "IdealDiode.sch" 50
+F2 "ID_in" B L 3825 1675 50
+F3 "ID_out" B R 4350 1775 50
+$EndSheet
+$Sheet
+S 4750 1625 525  200
+U 638DB850
+F0 "IdealDiode_USB" 50
+F1 "IdealDiode.sch" 50
+F2 "ID_in" B L 4750 1675 50
+F3 "ID_out" B R 5275 1775 50
+$EndSheet
+$Sheet
+S 5675 1625 525  200
+U 638DE946
+F0 "IdealDiode_5vreg" 50
+F1 "IdealDiode.sch" 50
+F2 "ID_in" B L 5675 1675 50
+F3 "ID_out" B R 6200 1775 50
+$EndSheet
+Text Label 4750 2700 0    50   ~ 0
+5v_USB
+Text Label 4750 1675 2    50   ~ 0
+5v_USB
+Text HLabel 5275 1775 2    50   Input ~ 0
+5VOUT
+Text HLabel 4350 1775 2    50   Input ~ 0
+5VOUT
+Text HLabel 6200 1775 2    50   Input ~ 0
+5VOUT
+Wire Wire Line
+	7900 3550 7900 3950
+Wire Wire Line
+	5450 2700 5450 3550
+Wire Wire Line
+	5450 3550 7900 3550
+Text Label 7350 4250 0    50   ~ 0
+5v_REG
+Text Label 5675 1675 2    50   ~ 0
+5v_REG
+Text HLabel 3150 2700 0    50   Input ~ 0
+USB_PWR
 $EndSCHEMATC

Commit message: Adapt 2590 board layout to ideal diodes and dual power input connector
Parts:
- R103, R104: footprint Resistors_SMD:R_0402 -> Resistor_SMD:R_0402_1005Metric
- U25: symbol smoothiev2-prime-rescue:BD47XXG-smoothieparts -> smoothiev2-prime-rescue:BD47XXG-smoothieparts-smoothiev2-prime-rescue
Connections:
- net labels added: 5V_PORTIN, USB_IN
- net labels removed: 5v_USB, USB_PWR
- wire segments 76 -> 79
Changed lines of the file:
@@
 $Descr A4 11693 8268
 encoding utf-8
-Sheet 10 13
+Sheet 6 13
 Title ""
 Date ""
@@
 UVLO
 $Comp
-L smoothiev2-prime-rescue:BD47XXG-smoothieparts U25
+L smoothiev2-prime-rescue:BD47XXG-smoothieparts-smoothiev2-prime-rescue U25
 U 1 1 627CE557
 P 2550 5800
@@
 F 0 "R104" H 3045 5846 50  0000 L CNN
 F 1 "7.1k" H 3045 5755 50  0000 L CNN
-F 2 "Resistors_SMD:R_0402" V 2905 5800 50  0001 C CNN
+F 2 "Resistor_SMD:R_0402_1005Metric" V 2905 5800 50  0001 C CNN
 F 3 "~" H 2975 5800 50  0001 C CNN
 	1    2975 5800
@@
 F 0 "R103" H 3045 5546 50  0000 L CNN
 F 1 "33k" H 3045 5455 50  0000 L CNN
-F 2 "Resistors_SMD:R_0402" V 2905 5500 50  0001 C CNN
+F 2 "Resistor_SMD:R_0402_1005Metric" V 2905 5500 50  0001 C CNN
 F 3 "~" H 2975 5500 50  0001 C CNN
 	1    2975 5500
@@
 Wire Notes Line
 	750  2150 9800 2150
-$Sheet
-S 3825 1625 525  200
-U 63881870
-F0 "IdealDiode" 50
-F1 "IdealDiode.sch" 50
-F2 "ID_in" B L 3825 1675 50
-F3 "ID_out" B R 4350 1775 50
-$EndSheet
-$Sheet
-S 4750 1625 525  200
-U 638DB850
-F0 "IdealDiode_USB" 50
-F1 "IdealDiode.sch" 50
-F2 "ID_in" B L 4750 1675 50
-F3 "ID_out" B R 5275 1775 50
-$EndSheet
 $Sheet
 S 5675 1625 525  200
@@
 F3 "ID_out" B R 6200 1775 50
 $EndSheet
-Text Label 4750 2700 0    50   ~ 0
-5v_USB
-Text Label 4750 1675 2    50   ~ 0
-5v_USB
 Text HLabel 5275 1775 2    50   Input ~ 0
-5VOUT
-Text HLabel 4350 1775 2    50   Input ~ 0
 5VOUT
 Text HLabel 6200 1775 2    50   Input ~ 0
@@
 Text Label 5675 1675 2    50   ~ 0
 5v_REG
-Text HLabel 3150 2700 0    50   Input ~ 0
-USB_PWR
+Text HLabel 4700 1450 0    50   Input ~ 0
+5V_PORTIN
+$Sheet
+S 4750 1625 525  200
+U 638DB850
+F0 "IdealDiode_USB" 50
+F1 "IdealDiode.sch" 50
+F2 "ID_in" B L 4750 1700 50
+F3 "ID_out" B R 5275 1775 50
+$EndSheet
+Wire Wire Line
+	4750 1700 4700 1700
+Wire Wire Line
+	4700 1700 4700 1450
+$Sheet
+S 3825 1625 525  200
+U 63881870
+F0 "IdealDiode" 50
+F1 "IdealDiode.sch" 50
+F2 "ID_in" B L 3825 1675 50
+F3 "ID_out" B R 4350 1750 50
+$EndSheet
+Text Label 4350 1750 0    50   ~ 0
+USB_IN
+Text Label 3150 2700 2    50   ~ 0
+USB_IN
+Wire Wire Line
+	4750 2700 5150 2700
+Connection ~ 4750 2700
+Connection ~ 5150 2700
 $EndSCHEMATC

Commit message: Updated 2660 version to match 2590 mods.
Updated 2660 version to match 2590 mods.  Ideal diodes, move board thermistor, add extra fet connector, modify probe input.
Parts:
- U25: symbol smoothiev2-prime-rescue:BD47XXG-smoothieparts-smoothiev2-prime-rescue -> smoothiev2-prime-2660-rescue:BD47XXG-smoothieparts-smoothiev2-prime-rescue-smoothiev2-prime-rescue
Changed lines of the file:
@@
 UVLO
 $Comp
-L smoothiev2-prime-rescue:BD47XXG-smoothieparts-smoothiev2-prime-rescue U25
+L smoothiev2-prime-2660-rescue:BD47XXG-smoothieparts-smoothiev2-prime-rescue-smoothiev2-prime-rescue U25
 U 1 1 627CE557
 P 2550 5800
