File: V2_Core_P1/V2 Core.kicad_pcb (KiCad board)
At the start: 4 copper layers, 90 x 110 mm, 340 parts, among them J1 USB_B, J10 Conn_01x02, J11 Conn_01x02, J12 Conn_01x02, J15 Conn_01x02, J16 Conn_01x02, J2 USB_A, J21 Conn_01x02, J22 Conn_01x02, J23 Conn_01x02, J24 Conn_01x03, J25 Conn_01x03, J26 Conn_01x03, J27 Conn_01x03, J28 Conn_01x03, J29 Conn_01x03, J3 Micro_SD_Card_Det, J30 Conn_01x03_Male, J32 Conn_02x05_Odd_Even, J33 Conn_02x05_Odd_Even, J34 Conn_02x05_Odd_Even, J35 Conn_02x05_Odd_Even, J36 Conn_02x05_Odd_Even, J37 Conn_02x05_Odd_Even, J38 Conn_02x05_Odd_Even, J39 Conn_02x05_Odd_Even, J4 RJ45_Hanrun_HR911105A, J40 Conn_02x05_Odd_Even, J41 Conn_ARM_JTAG_SWD_10, J42 Conn_01x02, J43 Conn_01x02, J44 Conn_01x02, J45 Conn_01x02, J5 Conn_02x20_Odd_Even, J6 Conn_01x03, J7 Conn_01x02, J8 Conn_01x02, J9 Conn_01x02, Q1 2N7002, Q2 2N7002, Q23 CJ2301 S1, Q24 CJ2301 S1, Q26 2N7002, Q27 MBT3906DW1, Q28 SQ3493EV, Q29 MBT3906DW1, Q3 2N7002, Q30 SQ3493EV, Q31 MBT3906DW1, Q32 SQ3493EV, Q4 WSD30L40DN, Q5 WSD3066DN33, Q6 2N7002, Q8 WSD3066DN33, SW1 SW_Push, SW2 TS-1185EC-C-D-B, U1 LAN8720A, U10 TPD4E1U06DCKR, U11 TPD4E1U06DCKR, U12 LMV324, U13 TPD4E1U06DCKR, U14 TPD4E1U06DCKR, U15 74LCX07, U16 MT9700, U17 TPD4E1U06DCKR, U18 MT9700, U19 MT9700, U2 STM32H745XIHx, U20 MT9700, U21 TPS5430DDA, U22 MT3410L, U23 AP22814AW5, U24 LMV331, U25 BD4722G, U4 AT25SF081-SSHF-X, U8 TPD4E1U06DCKR, U9 74HCT541, Y1 Crystal_GND24, Y2 Crystal, Y3 Crystal_GND24

Commit message: Minor position updates.
Parts:
- moved J5 0.15 mm to (186.3, 68.9)
Changed lines of the file:
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@@
 	(footprint "Connector_PinSocket_2.54mm:PinSocket_2x20_P2.54mm_Vertical"
 		(layer "F.Cu")
-		(at 186.14 68.93)
+		(at 186.29 68.93)
 		(descr "Through hole straight socket strip, 2x20, 2.54mm pitch, double cols (from Kicad 4.0.7), script generated")
 		(tags "Through hole socket strip THT 2x20 2.54mm double row")
@@
 	)
 	(segment
-		(start 178.75 71.440466)
-		(end 178.75 82.983345)
+		(start 184.91 93.1)
+		(end 186.14 94.33)
 		(width 0.2)
 		(layer "In1.Cu")
@@
 	)
 	(segment
-		(start 172.28 65.25)
-		(end 172.559534 65.25)
+		(start 172.559534 65.25)
+		(end 178.75 71.440466)
 		(width 0.2)
 		(layer "In1.Cu")
@@
 	)
 	(segment
-		(start 181.5 91.217351)
-		(end 183.182649 92.9)
+		(start 183.3 93.1)
+		(end 184.91 93.1)
 		(width 0.2)
 		(layer "In1.Cu")
@@
 	)
 	(segment
-		(start 183.182649 92.9)
-		(end 184.71 92.9)
+		(start 181.5 85.733345)
+		(end 181.5 91.217351)
 		(width 0.2)
 		(layer "In1.Cu")
@@
 	)
 	(segment
-		(start 181.5 85.733345)
-		(end 181.5 91.217351)
+		(start 182.129999 91.84735)
+		(end 182.129999 91.929999)
 		(width 0.2)
 		(layer "In1.Cu")
@@
 	)
 	(segment
-		(start 172.559534 65.25)
-		(end 178.75 71.440466)
+		(start 172.28 65.25)
+		(end 172.559534 65.25)
 		(width 0.2)
 		(layer "In1.Cu")
@@
 	)
 	(segment
-		(start 184.71 92.9)
-		(end 186.14 94.33)
+		(start 182.129999 91.929999)
+		(end 183.3 93.1)
+		(width 0.2)
+		(layer "In1.Cu")
+		(net 85)
+	)
+	(segment
+		(start 181.5 91.217351)
+		(end 182.129999 91.84735)
 		(width 0.2)
 		(layer "In1.Cu")
@@
 	)
 	(segment
+		(start 178.75 71.440466)
+		(end 178.75 82.983345)
+		(width 0.2)
+		(layer "In1.Cu")
+		(net 85)
+	)
+	(segment
 		(start 152.963348 53.909934)
 		(end 149.100568 53.909934)
@@
 	)
 	(segment
-		(start 181.8 91.984041)
-		(end 181.8 99.4)
+		(start 183.1 100.7)
+		(end 184.89 100.7)
 		(width 0.2)
 		(layer "In1.Cu")
@@
 	)
 	(segment
-		(start 181.8 99.4)
-		(end 182.9 100.5)
+		(start 181.17 85.92)
+		(end 181.17 91.354041)
 		(width 0.2)
 		(layer "In1.Cu")
@@
 	)
 	(segment
-		(start 182.9 100.5)
-		(end 184.69 100.5)
+		(start 181.8 91.984041)
+		(end 181.8 99.4)
 		(width 0.2)
 		(layer "In1.Cu")
@@
 	)
 	(segment
-		(start 184.69 100.5)
+		(start 184.89 100.7)
 		(end 186.14 101.95)
 		(width 0.2)
@@
 	)
 	(segment
-		(start 178.42 71.86)
-		(end 178.42 83.17)
+		(start 181.8 99.4)
+		(end 183.1 100.7)
 		(width 0.2)
 		(layer "In1.Cu")
@@
 	)
 	(segment
-		(start 181.17 85.92)
-		(end 181.17 91.354041)
+		(start 178.42 71.86)
+		(end 178.42 83.17)
 		(width 0.2)
 		(layer "In1.Cu")
@@
 	)
 	(segment
-		(start 172.81 66.25)
-		(end 178.42 71.86)
+		(start 181.17 91.354041)
+		(end 181.8 91.984041)
 		(width 0.2)
 		(layer "In1.Cu")
@@
 	)
 	(segment
-		(start 181.17 91.354041)
-		(end 181.8 91.984041)
+		(start 172.81 66.25)
+		(end 178.42 71.86)
 		(width 0.2)
 		(layer "In1.Cu")
@@
 	)
 	(segment
-		(start 117.725 117.8)
-		(end 117.6 117.675)
-		(width 1)
-		(layer "F.Cu")
-		(net 144)
-	)
-	(segment
 		(start 127.4 118.775)
 		(end 126.425 117.8)
@@
 	)
 	(segment
-		(start 117.6 117.675)
-		(end 117.6 114.7)
-		(width 1)
-		(layer "F.Cu")
-		(net 144)
-	)
-	(segment
 		(start 167.15 82.205)
 		(end 166.905 82.45)
@@
 	)
 	(segment
+		(start 118.0155 117.3155)
+		(end 118.0155 114.2845)
+		(width 2)
+		(layer "F.Cu")
+		(net 144)
+	)
+	(segment
 		(start 162.625998 77.01)
 		(end 163.485 77.01)
@@
 	)
 	(segment
+		(start 117.725 117.606)
+		(end 117.725 117.8)
+		(width 1)
+		(layer "F.Cu")
+		(net 144)
+	)
+	(segment
+		(start 118.0155 114.2845)
+		(end 119.25 113.05)
+		(width 2)
+		(layer "F.Cu")
+		(net 144)
+	)
+	(segment
 		(start 111.633 118.999)
 		(end 111.76 118.999)
@@
 	)
 	(segment
-		(start 117.6 114.7)
-		(end 119.25 113.05)
-		(width 2)
-		(layer "F.Cu")
-		(net 144)
-	)
-	(segment
 		(start 122.61 121.285)
 		(end 120.845 121.285)
@@
 		(layer "F.Cu")
 		(net 144)
+	)
+	(segment
+		(start 118.0155 117.3155)
+		(end 117.725 117.606)
+		(width 1)
+		(layer "F.Cu")
+		(net 144)
